File: stepdown-lowpower.kicad_pcb (KiCad board)
At the start: 2 copper layers, 61 x 49.5 mm, 15 parts, among them J1 Output_Screw_Terminal, J2 Input_Screw_Terminal, U1 VXO78012-1000, U2 VXO7803-1000

Commit message: Silkscreen update
Other:
- board text added: "StepDown LowPower V1.2 2022-09-08"
- board text removed: "LowPower StepDown 2022-09-08"
Changed lines of the file:
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@@
     (effects (font (size 1 1) (thickness 0.15)))
   )
-  (gr_text "LowPower StepDown\n2022-09-08" (at 72.39 76.2) (layer "F.SilkS")
+  (gr_text "StepDown LowPower\nV1.2\n2022-09-08" (at 72.39 76.2) (layer "F.SilkS")
     (effects (font (size 1 1) (thickness 0.15)))
   )
